File: KiCad_HHKB-JP_Poker.kicad_sch (KiCad schematic)
At the start: 21 parts, among them SW1 SW_Push, U1 ATmega32U4-MU, U2 PRTR5V0U2X, Y1 16MHz

Commit message: Modify Symbol Name
Other:
- moved on the sheet: C1, C2, C3, C4, D32, F1, L1, R2, R6, U2, USB1
