File: matrix.kicad_sch (KiCad schematic)
At the start: 132 parts

Commit message: 回路図エディターで COL14削除、結局 JP60から、 ]と backspace の位置だけ変更した
Parts:
- renumbered K_UNSC1 to K_BKSL1, K_PIPE1 to K_YEN1
Connections:
- net COL14 is gone; now on net COL13: K_BKSPC1.1 (COL)
- net ROW0: no longer D17.1 (K)
- net ROW1: now also D17.1 (K)
Other:
- moved on the sheet: D17, K_BKSPC1
Changed lines of the file:
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@@
   (junction (at 169.545 94.615) (diameter 0) (color 0 0 0 0)
   )
+  (junction (at 217.805 78.74) (diameter 0) (color 0 0 0 0)
+  )
   (junction (at 212.725 52.705) (diameter 0) (color 0 0 0 0)
   )
@@
   (junction (at 205.74 94.615) (diameter 0) (color 0 0 0 0)
   )
-  (junction (at 229.87 62.865) (diameter 0) (color 0 0 0 0)
-  )
   (junction (at 116.205 68.58) (diameter 0) (color 0 0 0 0)
   )
@@
   (junction (at 133.35 62.865) (diameter 0) (color 0 0 0 0)
   )
+  (junction (at 236.855 68.58) (diameter 0) (color 0 0 0 0)
+  )
   (wire (pts (xy 157.48 57.785) (xy 159.385 57.785))
     (stroke (width 0) (type default) (color 0 0 0 0))
   )
+  (wire (pts (xy 217.805 78.74) (xy 229.87 78.74))
+    (stroke (width 0) (type default) (color 0 0 0 0))
+  )
   (wire (pts (xy 97.155 121.285) (xy 99.06 121.285))
     (stroke (width 0) (type default) (color 0 0 0 0))
@@
     (stroke (width 0) (type default) (color 0 0 0 0))
   )
-  (wire (pts (xy 248.92 36.83) (xy 248.92 52.705))
-    (stroke (width 0) (type default) (color 0 0 0 0))
-  )
   (wire (pts (xy 157.48 105.41) (xy 159.385 105.41))
     (stroke (width 0) (type default) (color 0 0 0 0))
@@
     (stroke (width 0) (type default) (color 0 0 0 0))
   )
+  (wire (pts (xy 236.855 68.58) (xy 236.855 84.455))
+    (stroke (width 0) (type default) (color 0 0 0 0))
+  )
   (wire (pts (xy 176.53 52.705) (xy 176.53 36.83))
     (stroke (width 0) (type default) (color 0 0 0 0))
@@
     (stroke (width 0) (type default) (color 0 0 0 0))
   )
-  (wire (pts (xy 229.87 62.865) (xy 241.935 62.865))
-    (stroke (width 0) (type default) (color 0 0 0 0))
-  )
   (wire (pts (xy 73.025 89.535) (xy 74.93 89.535))
     (stroke (width 0) (type default) (color 0 0 0 0))
   )
-  (wire (pts (xy 241.935 57.785) (xy 243.84 57.785))
+  (wire (pts (xy 229.87 73.66) (xy 231.775 73.66))
     (stroke (width 0) (type default) (color 0 0 0 0))
   )
@@
     (stroke (width 0) (type default) (color 0 0 0 0))
   )
-  (wire (pts (xy 236.855 52.705) (xy 236.855 84.455))
+  (wire (pts (xy 236.855 52.705) (xy 236.855 68.58))
     (stroke (width 0) (type default) (color 0 0 0 0))
   )
@@
     )
   )
-  (global_label "COL14" (shape input) (at 248.92 36.83 180) (fields_autoplaced)
-    (effects (font (size 1.27 1.27)) (justify right))
-    (property "Intersheet References" "${INTERSHEET_REFS}" (id 0) (at 240.5482 36.7506 0)
-      (effects (font (size 1.27 1.27)) (justify right) hide)
-    )
-  )
   (global_label "COL10" (shape input) (at 200.66 36.83 180) (fields_autoplaced)
     (effects (font (size 1.27 1.27)) (justify right))
@@
   (symbol (lib_id "MX_Alps_Hybrid:MX-NoLED") (at 233.045 53.975 0) (unit 1)
     (in_bom yes) (on_board yes)
-    (property "Reference" "K_PIPE1" (id 0) (at 233.8832 48.3108 0)
+    (property "Reference" "K_YEN1" (id 0) (at 233.8832 48.3108 0)
       (effects (font (size 1.524 1.524)))
     )
@@
     (pin "2")
   )
-  (symbol (lib_id "MX_Alps_Hybrid:MX-NoLED") (at 245.11 53.975 0) (unit 1)
-    (in_bom yes) (on_board yes)
-    (property "Reference" "K_BKSPC1" (id 0) (at 245.9482 48.3108 0)
-      (effects (font (size 1.524 1.524)))
-    )
-    (property "Value" "MX-NoLED" (id 1) (at 245.9482 50.1904 0)
-      (effects (font (size 0.508 0.508)))
-    )
-    (property "Footprint" "MX_Only:MXOnly-1U-Hotswap" (id 2) (at 229.235 54.61 0)
-      (effects (font (size 1.524 1.524)) hide)
-    )
-    (property "Datasheet" "" (id 3) (at 229.235 54.61 0)
-      (effects (font (size 1.524 1.524)) hide)
-    )
-    (pin "1")
-    (pin "2")
-  )
-  (symbol (lib_id "Device:D_Small") (at 241.935 60.325 90) (unit 1)
-    (in_bom yes) (on_board yes)
-    (property "Reference" "D17" (id 0) (at 243.6622 59.1566 90)
-      (effects (font (size 1.27 1.27)) (justify right))
-    )
-    (property "Value" "SOD-123" (id 1) (at 243.6622 61.468 90)
-      (effects (font (size 1.27 1.27)) (justify right))
-    )
-    (property "Footprint" "Diode_SMD:D_SOD-123" (id 2) (at 241.935 60.325 90)
-      (effects (font (size 1.27 1.27)) hide)
-    )
-    (property "Datasheet" "~" (id 3) (at 241.935 60.325 90)
+  (symbol (lib_id "MX_Alps_Hybrid:MX-NoLED") (at 233.045 69.85 0) (unit 1)
+    (in_bom yes) (on_board yes)
+    (property "Reference" "K_BKSPC1" (id 0) (at 233.8832 64.1858 0)
+      (effects (font (size 1.524 1.524)))
+    )
+    (property "Value" "MX-NoLED" (id 1) (at 233.8832 66.0654 0)
+      (effects (font (size 0.508 0.508)))
+    )
+    (property "Footprint" "MX_Only:MXOnly-1U-Hotswap" (id 2) (at 217.17 70.485 0)
+      (effects (font (size 1.524 1.524)) hide)
+    )
+    (property "Datasheet" "" (id 3) (at 217.17 70.485 0)
+      (effects (font (size 1.524 1.524)) hide)
+    )
+    (pin "1")
+    (pin "2")
+  )
+  (symbol (lib_id "Device:D_Small") (at 229.87 76.2 90) (unit 1)
+    (in_bom yes) (on_board yes)
+    (property "Reference" "D17" (id 0) (at 231.5972 75.0316 90)
+      (effects (font (size 1.27 1.27)) (justify right))
+    )
+    (property "Value" "SOD-123" (id 1) (at 231.5972 77.343 90)
+      (effects (font (size 1.27 1.27)) (justify right))
+    )
+    (property "Footprint" "Diode_SMD:D_SOD-123" (id 2) (at 229.87 76.2 90)
+      (effects (font (size 1.27 1.27)) hide)
+    )
+    (property "Datasheet" "~" (id 3) (at 229.87 76.2 90)
       (effects (font (size 1.27 1.27)) hide)
     )
@@
   (symbol (lib_id "MX_Alps_Hybrid:MX-NoLED") (at 208.915 101.6 0) (unit 1)
     (in_bom yes) (on_board yes)
-    (property "Reference" "K_UNSC1" (id 0) (at 209.7532 95.9358 0)
-      (effects (font (size 1.524 1.524)))
-    )
+    (property "Reference" "K_BKSL1" (id 0) (at 209.7532 95.9358 0)
+      (effects (font (size 1.524 1.524)))
+    )

Commit message: 縦（Col）の配線完了
Parts:
- renumbered D15 to D10, D12 to D11, D13 to D12, D14 to D13, D21 to D14, D16 to D15, D18 to D16, D19 to D17, D20 to D18, D26 to D19, D1 to D20, D23 to D21, D24 to D22, D25 to D23, D31 to D24, D10 to D25, D28 to D26, D29 to D27, D30 to D28, D36 to D29, D11 to D30, D37 to D31, D33 to D32, D34 to D33, D35 to D34, D41 to D35, D42 to D36, D38 to D37, D39 to D38, D40 to D39, D47 to D40, D44 to D41, D45 to D42, D46 to D43, D52 to D44, D49 to D45, D50 to D46, D51 to D47, D57 to D48, D54 to D49, D55 to D50, D56 to D51, D62 to D52, D59 to D53, D60 to D54, D61 to D55, D22 to D56, D63 to D57, D65 to D58, D66 to D59, D71 to D60, D43 to D61, D27 to D62, D70 to D63, D17 to D64, D72 to D65, D67 to D66, D74 to D67, K_]2 to K_]1
