File: matrix.kicad_sch (KiCad schematic)
At the start: 132 parts

Commit message: 検算完了！完成！
Parts:
- K_RIGHT1: footprint MX_Only:MXOnly-1.25U-Hotswap -> MX_Only:MXOnly-1U-Hotswap
Changed lines of the file:
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@@
       (effects (font (size 0.508 0.508)))
     )
-    (property "Footprint" "MX_Only:MXOnly-1.25U-Hotswap" (id 2) (at 217.17 118.11 0)
+    (property "Footprint" "MX_Only:MXOnly-1U-Hotswap" (id 2) (at 217.17 118.11 0)
       (effects (font (size 1.524 1.524)) hide)
     )
