File: PCB_Plate/KiCad_KMKB-JP_Poker.kicad_pcb (KiCad board)
At the start: 2 copper layers, 285 x 95.1 mm, 155 parts, among them SW1 SW_Push, U1 ATmega32U4-MU, U2 PRTR5V0U2X, Y1 16MHz

Commit message: ドーターボード用の配線穴を設置
Parts:
- added J1: Conn_01x04, Connector_PinHeader_2.54mm:PinHeader_1x04_P2.54mm_Vertical, F.Cu at (128.4, 200.4)
Routing:
- net VCC: track 38.2 -> 65.1 mm
- net D+: track 88.1 -> 114.8 mm, vias 0 -> 1
- net D-: track 87.2 -> 113.5 mm, vias 0 -> 1
- net GND: track 213.2 -> 235.4 mm
- net COL0: track 113.7 -> 108.1 mm, vias 7 -> 2
Other:
- board text added: "D-"
- board text added: "GND"
- board text added: "VCC"

Commit message: ドーターボード用の配線穴の位置を微修正
Parts:
- moved J1 5.72 mm to (128.3, 206.1)
Routing:
- net VCC: track 65.1 -> 70.8 mm
- net GND: track 235.4 -> 241.1 mm
- net D+: track 114.8 -> 109.8 mm
- net D-: track 113.5 -> 108.4 mm
Changed lines of the file:
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@@
   )
   (footprint "Connector_PinHeader_2.54mm:PinHeader_1x04_P2.54mm_Vertical" (layer "F.Cu")
-    (at 128.397 200.396 180)
+    (at 128.27 206.111 180)
     (descr "Through hole straight pin header, 1x04, 2.54mm pitch, single row")
     (tags "Through hole pin header THT 1x04 2.54mm single row")
@@
   (segment (start 146.431 180.213) (end 146.431 181.102) (width 0.381) (layer "B.Cu") (net 75))
   (segment (start 166.409375 255.46875) (end 164.409375 257.46875) (width 0.381) (layer "B.Cu") (net 75))
+  (segment (start 134.874 178.3335) (end 129.5145 178.3335) (width 0.381) (layer "B.Cu") (net 75))
   (segment (start 145.923 189.23) (end 153.162 189.23) (width 0.381) (layer "B.Cu") (net 75))
   (segment (start 136.779 179.451) (end 136.779 178.3335) (width 0.381) (layer "B.Cu") (net 75))
@@
   (segment (start 163.409375 258.46875) (end 164.409375 257.46875) (width 0.381) (layer "B.Cu") (net 75))
   (segment (start 161.071875 258.46875) (end 159.535875 258.46875) (width 0.254) (layer "B.Cu") (net 75))
-  (segment (start 129.5145 178.3335) (end 134.874 178.3335) (width 0.381) (layer "B.Cu") (net 75))
   (segment (start 158.996875 260.27775) (end 158.488875 260.78575) (width 0.254) (layer "B.Cu") (net 75))
   (segment (start 161.909375 254.13125) (end 161.909375 254.7511) (width 0.254) (layer "B.Cu") (net 75))
-  (segment (start 126.111 181.737) (end 129.5145 178.3335) (width 0.381) (layer "B.Cu") (net 75))
   (segment (start 153.162 189.23) (end 153.67 189.738) (width 0.381) (layer "B.Cu") (net 75))
   (segment (start 139.9675 179.5645) (end 139.573 179.959) (width 0.381) (layer "B.Cu") (net 75))
@@
   (segment (start 139.573 179.959) (end 137.287 179.959) (width 0.381) (layer "B.Cu") (net 75))
   (segment (start 152.646875 260.78575) (end 151.986375 260.12525) (width 0.254) (layer "B.Cu") (net 75))
+  (segment (start 126.111 196.332) (end 128.27 198.491) (width 0.381) (layer "B.Cu") (net 75))
   (segment (start 139.573 179.959) (end 139.827 180.213) (width 0.381) (layer "B.Cu") (net 75))
   (segment (start 157.701375 261.01425) (end 157.472875 260.78575) (width 0.254) (layer "B.Cu") (net 75))
   (segment (start 168.783 189.738) (end 168.91 189.865) (width 0.381) (layer "B.Cu") (net 75))
+  (segment (start 129.5145 178.3335) (end 126.111 181.737) (width 0.381) (layer "B.Cu") (net 75))
   (segment (start 153.67 189.738) (end 168.783 189.738) (width 0.381) (layer "B.Cu") (net 75))
   (segment (start 178.21475 258.732) (end 184.51475 258.732) (width 0.381) (layer "B.Cu") (net 75))
@@
   (segment (start 167.746875 255.46875) (end 169.355875 255.46875) (width 0.254) (layer "B.Cu") (net 75))
   (segment (start 167.746875 259.46875) (end 166.409375 259.46875) (width 0.254) (layer "B.Cu") (net 75))
-  (segment (start 126.111 190.49) (end 126.111 181.737) (width 0.381) (layer "B.Cu") (net 75))
+  (segment (start 126.111 181.737) (end 126.111 196.332) (width 0.381) (layer "B.Cu") (net 75))
   (segment (start 159.535875 258.46875) (end 158.996875 259.00775) (width 0.254) (layer "B.Cu") (net 75))
   (segment (start 169.355875 255.46875) (end 169.918875 254.90575) (width 0.254) (layer "B.Cu") (net 75))
@@
   (segment (start 164.409375 257.2003) (end 164.409375 257.46875) (width 0.381) (layer "B.Cu") (net 75))
   (segment (start 154.361375 257.73775) (end 152.011875 257.73775) (width 0.254) (layer "B.Cu") (net 75))
-  (segment (start 128.397 192.776) (end 126.111 190.49) (width 0.381) (layer "B.Cu") (net 75))
-  (segment (start 130.195837 196.818157) (end 129.434843 196.818157) (width 0.261112) (layer "F.Cu") (net 76))
   (segment (start 147.417025 205.911344) (end 146.969837 205.464156) (width 0.261112) (layer "F.Cu") (net 76))
-  (segment (start 129.434843 196.818157) (end 128.397 197.856) (width 0.261112) (layer "F.Cu") (net 76))
-  (segment (start 131.212844 197.835164) (end 130.195837 196.818157) (width 0.261112) (layer "F.Cu") (net 76))
-  (segment (start 146.969837 205.464156) (end 134.015836 205.464156) (width 0.261112) (layer "F.Cu") (net 76))
-  (segment (start 134.015836 205.464156) (end 131.212844 202.661164) (width 0.261112) (layer "F.Cu") (net 76))
+  (segment (start 130.703837 202.533157) (end 129.307843 202.533157) (width 0.261112) (layer "F.Cu") (net 76))
   (segment (start 147.417025 206.150975) (end 147.417025 205.911344) (width 0.261112) (layer "F.Cu") (net 76))
-  (segment (start 131.212844 202.661164) (end 131.212844 197.835164) (width 0.261112) (layer "F.Cu") (net 76))
+  (segment (start 133.634836 205.464156) (end 130.703837 202.533157) (width 0.261112) (layer "F.Cu") (net 76))
+  (segment (start 146.969837 205.464156) (end 133.634836 205.464156) (width 0.261112) (layer "F.Cu") (net 76))
+  (segment (start 129.307843 202.533157) (end 128.27 203.571) (width 0.261112) (layer "F.Cu") (net 76))
   (via (at 147.417025 206.150975) (size 0.6) (drill 0.4) (layers "F.Cu" "B.Cu") (net 76))
   (segment (start 146.706844 197.388836) (end 146.706844 194.152164) (width 0.261112) (layer "B.Cu") (net 76))
@@
   (segment (start 151.659844 241.711836) (end 151.659844 210.154164) (width 0.261112) (layer "B.Cu") (net 76))
   (segment (start 143.785844 190.870844) (end 143.018 190.103) (width 0.261112) (layer "B.Cu") (net 76))
+  (segment (start 133.827164 204.999844) (end 130.896163 202.068843) (width 0.261112) (layer "F.Cu") (net 77))
+  (segment (start 147.162163 204.999844) (end 133.827164 204.999844) (width 0.261112) (layer "F.Cu") (net 77))
+  (segment (start 130.896163 202.068843) (end 129.307843 202.068843) (width 0.261112) (layer "F.Cu") (net 77))
   (segment (start 147.984975 205.583025) (end 147.745344 205.583025) (width 0.261112) (layer "F.Cu") (net 77))
-  (segment (start 129.434843 196.353843) (end 128.397 195.316) (width 0.261112) (layer "F.Cu") (net 77))
-  (segment (start 131.677156 202.468836) (end 131.677156 197.642836) (width 0.261112) (layer "F.Cu") (net 77))
-  (segment (start 131.677156 197.642836) (end 130.388163 196.353843) (width 0.261112) (layer "F.Cu") (net 77))
-  (segment (start 147.162163 204.999844) (end 134.208164 204.999844) (width 0.261112) (layer "F.Cu") (net 77))
   (segment (start 147.745344 205.583025) (end 147.162163 204.999844) (width 0.261112) (layer "F.Cu") (net 77))
-  (segment (start 134.208164 204.999844) (end 131.677156 202.468836) (width 0.261112) (layer "F.Cu") (net 77))
-  (segment (start 130.388163 196.353843) (end 129.434843 196.353843) (width 0.261112) (layer "F.Cu") (net 77))
+  (segment (start 129.307843 202.068843) (end 128.27 201.031) (width 0.261112) (layer "F.Cu") (net 77))
   (via (at 147.984975 205.583025) (size 0.6) (drill 0.4) (layers "F.Cu" "B.Cu") (net 77))
   (segment (start 146.028156 198.724164) (end 147.171156 197.581164) (width 0.261112) (layer "B.Cu") (net 77))
@@
   (segment (start 144.653 189.103) (end 141.986 189.103) (width 0.381) (layer "F.Cu") (net 98))
   (segment (start 145.923 181.864) (end 142.24 181.864) (width 0.381) (layer "F.Cu") (net 98))
-  (segment (start 128.143 189.103) (end 141.986 189.103) (width 0.381) (layer "F.Cu") (net 98))
+  (segment (start 126.111 203.952) (end 128.27 206.111) (width 0.381) (layer "F.Cu") (net 98))
   (segment (start 148.082 179.451) (end 149.606 180.975) (width 0.381) (layer "F.Cu") (net 98))
   (segment (start 145.542 180.213) (end 145.542 179.959) (width 0.381) (layer "F.Cu") (net 98))
+  (segment (start 128.143 189.103) (end 126.111 191.135) (width 0.381) (layer "F.Cu") (net 98))
   (segment (start 146.05 179.451) (end 148.082 179.451) (width 0.381) (layer "F.Cu") (net 98))
   (segment (start 149.606 180.975) (end 149.606 182.499) (width 0.381) (layer "F.Cu") (net 98))
   (segment (start 147.828 192.278) (end 144.653 189.103) (width 0.381) (layer "F.Cu") (net 98))
-  (segment (start 126.238 198.237) (end 126.238 191.008) (width 0.381) (layer "F.Cu") (net 98))
+  (segment (start 126.111 191.135) (end 126.111 203.952) (width 0.381) (layer "F.Cu") (net 98))
+  (segment (start 141.986 189.103) (end 128.143 189.103) (width 0.381) (layer "F.Cu") (net 98))
   (segment (start 142.24 181.864) (end 142.113 181.991) (width 0.381) (layer "F.Cu") (net 98))
   (segment (start 149.606 182.499) (end 148.844 183.261) (width 0.381) (layer "F.Cu") (net 98))
-  (segment (start 128.397 200.396) (end 126.238 198.237) (width 0.381) (layer "F.Cu") (net 98))
-  (segment (start 126.238 191.008) (end 128.143 189.103) (width 0.381) (layer "F.Cu") (net 98))
   (segment (start 148.844 183.261) (end 147.32 183.261) (width 0.381) (layer "F.Cu") (net 98))
   (segment (start 147.32 183.261) (end 145.923 181.864) (width 0.381) (layer "F.Cu") (net 98))

Commit message: シルクを修正
Other:
- board text added: "D+"
Changed lines of the file:
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@@
   (gr_circle (center 155.58135 231.9274) (end 158.08135 231.9274) (layer "B.SilkS") (width 0.15) (fill none))
   (gr_line (start 174.498 212.598) (end 161.13125 212.598) (layer "Cmts.User") (width 0.15))
-  (gr_text "GND" (at 128.016 203.2) (layer "B.SilkS")
+  (gr_text "GND" (at 128.27 195.453) (layer "B.SilkS")
     (effects (font (size 1.5 1.5) (thickness 0.3)) (justify mirror))
   )
   (gr_text "2U" (at 143.66875 242.09375) (layer "B.SilkS")
     (effects (font (size 1 1) (thickness 0.15)) (justify mirror))
+  )
+  (gr_text "D+" (at 131.064 201.041) (layer "B.SilkS")
+    (effects (font (size 1.5 1.5) (thickness 0.3)) (justify mirror))
   )
   (gr_text "ISO-ENTER" (at 395.2875 210.34375 270) (layer "B.SilkS")
@@
     (effects (font (size 1 1) (thickness 0.15)) (justify mirror))
   )
-  (gr_text "D-\n" (at 131.318 195.326) (layer "B.SilkS")
+  (gr_text "D-\n" (at 131.064 203.581) (layer "B.SilkS")
     (effects (font (size 1.5 1.5) (thickness 0.3)) (justify mirror))
   )
@@
     (effects (font (size 1 1) (thickness 0.15)) (justify mirror))
   )
-  (gr_text "VCC" (at 131.572 192.786) (layer "B.SilkS")
+  (gr_text "VCC" (at 128.143 208.788) (layer "B.SilkS")
     (effects (font (size 1.5 1.5) (thickness 0.3)) (justify mirror))
   )

Commit message: JCLPCBに発注しました
Routing:
- net VCC: track 70.8 -> 72.5 mm
Changed lines of the file:
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@@
     (solder_mask_min_width 0.25)
     (pcbplotparams
-      (layerselection 0x00010fc_ffffffff)
+      (layerselection 0x00010f0_ffffffff)
       (disableapertmacros false)
-      (usegerberextensions true)
+      (usegerberextensions false)
       (usegerberattributes false)
       (usegerberadvancedattributes false)
@@
       (plotinvisibletext false)
       (sketchpadsonfab false)
-      (subtractmaskfromsilk true)
+      (subtractmaskfromsilk false)
       (outputformat 1)
       (mirror false)
       (drillshape 0)
       (scaleselection 1)
-      (outputdirectory "Gerber/")
+      (outputdirectory "C:/Users/scbp6/Documents/KiCad/6.0/projects/KiCad_KMKB-JP_Poker/PCB_Plate/Files_for_production/Gerber/")
     )
   )
@@
     (pad "44" smd roundrect locked (at -2.5 3.3375 90) (size 0.25 1.075) (layers "B.Cu" "B.Paste" "B.Mask") (roundrect_rratio 0.25)
       (net 2 "+5V") (pinfunction "AVCC") (pintype "passive"))
-    (pad "45" smd roundrect locked (at 0 0 90) (size 5.2 5.2) (layers "B.Cu" "B.Mask") (roundrect_rratio 0.048077)
+    (pad "45" smd roundrect locked (at 0 0 90) (size 5.2 5.2) (layers "B.Cu" "B.Mask") (roundrect_rratio 0.04807692308)
       (net 75 "GND") (pinfunction "GND") (pintype "passive"))
     (model "${KISYS3DMOD}/Package_DFN_QFN.3dshapes/QFN-44-1EP_7x7mm_P0.5mm_EP5.2x5.2mm.wrl"
@@
   (segment (start 178.08575 234.15625) (end 178.08575 233.83875) (width 0.254) (layer "B.Cu") (net 97))
   (segment (start 144.653 189.103) (end 141.986 189.103) (width 0.381) (layer "F.Cu") (net 98))
-  (segment (start 145.923 181.864) (end 142.24 181.864) (width 0.381) (layer "F.Cu") (net 98))
+  (segment (start 149.225 183.642) (end 146.939 183.642) (width 0.381) (layer "F.Cu") (net 98))
   (segment (start 126.111 203.952) (end 128.27 206.111) (width 0.381) (layer "F.Cu") (net 98))
-  (segment (start 148.082 179.451) (end 149.606 180.975) (width 0.381) (layer "F.Cu") (net 98))
-  (segment (start 145.542 180.213) (end 145.542 179.959) (width 0.381) (layer "F.Cu") (net 98))
+  (segment (start 148.844 179.451) (end 150.114 180.721) (width 0.381) (layer "F.Cu") (net 98))
   (segment (start 128.143 189.103) (end 126.111 191.135) (width 0.381) (layer "F.Cu") (net 98))
-  (segment (start 146.05 179.451) (end 148.082 179.451) (width 0.381) (layer "F.Cu") (net 98))
-  (segment (start 149.606 180.975) (end 149.606 182.499) (width 0.381) (layer "F.Cu") (net 98))
+  (segment (start 146.05 179.451) (end 148.844 179.451) (width 0.381) (layer "F.Cu") (net 98))
   (segment (start 147.828 192.278) (end 144.653 189.103) (width 0.381) (layer "F.Cu") (net 98))
+  (segment (start 142.24 181.864) (end 142.113 181.991) (width 0.381) (layer "F.Cu") (net 98))
   (segment (start 126.111 191.135) (end 126.111 203.952) (width 0.381) (layer "F.Cu") (net 98))
+  (segment (start 145.161 181.864) (end 142.24 181.864) (width 0.381) (layer "F.Cu") (net 98))
   (segment (start 141.986 189.103) (end 128.143 189.103) (width 0.381) (layer "F.Cu") (net 98))
-  (segment (start 142.24 181.864) (end 142.113 181.991) (width 0.381) (layer "F.Cu") (net 98))
-  (segment (start 149.606 182.499) (end 148.844 183.261) (width 0.381) (layer "F.Cu") (net 98))
-  (segment (start 148.844 183.261) (end 147.32 183.261) (width 0.381) (layer "F.Cu") (net 98))
-  (segment (start 147.32 183.261) (end 145.923 181.864) (width 0.381) (layer "F.Cu") (net 98))
+  (segment (start 146.939 183.642) (end 145.161 181.864) (width 0.381) (layer "F.Cu") (net 98))
+  (segment (start 150.114 182.753) (end 149.225 183.642) (width 0.381) (layer "F.Cu") (net 98))
   (segment (start 145.542 179.959) (end 146.05 179.451) (width 0.381) (layer "F.Cu") (net 98))
+  (segment (start 150.114 180.721) (end 150.114 182.753) (width 0.381) (layer "F.Cu") (net 98))
+  (segment (start 145.542 180.213) (end 145.542 179.959) (width 0.381) (layer "F.Cu") (net 98))
   (via (at 147.828 192.278) (size 0.6) (drill 0.4) (layers "F.Cu" "B.Cu") (net 98))
   (via (at 145.542 180.213) (size 0.6) (drill 0.4) (layers "F.Cu" "B.Cu") (net 98))
