File: TOP_Plate/Poker/matrix.kicad_sch (KiCad schematic)
At the start: 132 parts

Commit message: SAVE POINT
Parts:
- D10, D11, D12, D13, D14, D15, D16, D17, D18, D19, D2, D20, D21, D22, D23, D24, D25, D26, D27, D28, D29, D3, D30, D31, D32, D33, D34, D35, D36, D37, D38, D39, D4, D40, D41, D42, D43, D44, D45, D46, D47, D48, D49, D5, D50, D51, D52, D53, D54, D55, D56, D57, D58, D59, D6, D60, D61, D62, D63, D64, D65, D66, D67, D7, D8, D9: footprint Diode_SMD:D_SOD-123 -> (none)
- K_#0_1, K_#1, K_#2, K_#3, K_#4, K_#5, K_#6, K_#7, K_#8, K_#9, K_,1, K_-1, K_.1, K_/1, K_:1, K_;1, K_=1, K_@1, K_A1, K_B1, K_BKSL1, K_BKSPC1, K_C1, K_D1, K_DOWN1, K_E1, K_ESC1, K_F1, K_G1, K_H1, K_HENK1, K_I1, K_J1, K_K1, K_L1, K_LALT1, K_LCTRL1, K_LEFT1, K_M1, K_N1, K_NHENK1, K_O1, K_P1, K_Q1, K_R1, K_RIGHT1, K_RSFT1, K_S1, K_T1, K_U1, K_UP1, K_V1, K_W1, K_WIN1, K_X1, K_Y1, K_YEN1, K_Z1, K_[1, K_]1: footprint MX_Only:MXOnly-1U-Hotswap -> kbd_SW_Hole:SW_Hole_1u
- K_CAPS1: footprint MX_Only:MXOnly-1.75U-Hotswap -> kbd_SW_Hole:SW_Hole_TH_1.75u
- K_ENTER1: footprint MX_Only:MXOnly-ISO-ROTATED-Hotswap -> kbd_SW_Hole:SW_Hole_2u
- K_LSFT1: footprint MX_Only:MXOnly-2U-Hotswap -> kbd_SW_Hole:SW_Hole_TH_2u
- K_LSPACE1, K_RSPACE1: footprint MX_Only:MXOnly-1.25U-Hotswap -> kbd_SW_Hole:SW_Hole_1.25u
- K_TAB1: footprint MX_Only:MXOnly-1.5U-Hotswap -> kbd_SW_Hole:SW_Hole_1.5u
