File: TOP_Plate/Poker/KMKB-JP_Poker_SwitchPlate.kicad_pcb (KiCad board)
At the start: 2 copper layers, 285 x 95.1 mm, 156 parts, among them J1 Conn_01x04, SW1 SW_Push, U1 ATmega32U4-MU, U2 PRTR5V0U2X, Y1 16MHz

Commit message: SAVE POINT
Parts:
- removed C1, C2: 22pF, Capacitor_SMD:C_0603_1608Metric
- removed C3: 1uF, Capacitor_SMD:C_0603_1608Metric
- removed C4, C5, C6: 0.1uF, Capacitor_SMD:C_0603_1608Metric
- removed C7: 10uF, Capacitor_SMD:C_0603_1608Metric
- removed D1: SMF6.0CA, Diode_SMD:D_SOD-123
- removed D10, D11, D12, D13, D14, D15, D16, D17, D18, D19, D2, D20, D21, D22, D23, D24, D25, D26, D27, D28, D29, D3, D30, D31, D32, D33, D34, D35, D36, D37, D38, D39, D4, D40, D41, D42, D43, D44, D45, D46, D47, D48, D49, D5, D50, D51, D52, D53, D54, D55, D56, D57, D58, D59, D6, D60, D61, D62, D63, D64, D65, D66, D67, D7, D8, D9: SOD-123, Diode_SMD:D_SOD-123
- removed F1: Polyfuse_Small, Fuse:Fuse_1206_3216Metric
- removed G***: LOGO, kuzumotch_icon:kuzumotch_icon
- removed J1: Conn_01x04, Connector_PinHeader_2.54mm:PinHeader_1x04_P2.54mm_Vertical
- removed L1: 60R@100MHz, Inductor_SMD:L_1206_3216Metric
- removed R1, R2: 22, Resistor_SMD:R_0603_1608Metric
- removed R3: 10k, Resistor_SMD:R_0603_1608Metric
- removed R4, R5: 5.1k, Resistor_SMD:R_0603_1608Metric
- removed R6: 1k, Resistor_SMD:R_0603_1608Metric
- removed REF**: 60_Outline, locallib:60_Outline-Modded-Extreme-deleteCenterHole
- removed SW1: SW_Push, Button_Switch_SMD:SW_SPST_TL3342
- removed U1: ATmega32U4-MU, Package_DFN_QFN:QFN-44-1EP_7x7mm_P0.5mm_EP5.2x5.2mm
- removed U2: PRTR5V0U2X, random-keyboard-parts:SOT143B
- removed USB1: HRO-TYPE-C-31-M-12, Type-C:HRO-TYPE-C-31-M-12-Assembly
- removed Y1: 16MHz, Crystal:Crystal_SMD_3225-4Pin_3.2x2.5mm
- added K_#0_1: MX-NoLED, kbd_SW_Hole:SW_Hole_1u, F.Cu at (479.6, 44.2)
- added K_#1: MX-NoLED, kbd_SW_Hole:SW_Hole_1u, F.Cu at (308.1, 44.2)
- added K_#2: MX-NoLED, kbd_SW_Hole:SW_Hole_1u, F.Cu at (327.2, 44.2)
- added K_#3: MX-NoLED, kbd_SW_Hole:SW_Hole_1u, F.Cu at (346.2, 44.2)
- added K_#4: MX-NoLED, kbd_SW_Hole:SW_Hole_1u, F.Cu at (365.3, 44.2)
- added K_#5: MX-NoLED, kbd_SW_Hole:SW_Hole_1u, F.Cu at (384.3, 44.2)
- added K_#6: MX-NoLED, kbd_SW_Hole:SW_Hole_1u, F.Cu at (403.4, 44.2)
- added K_#7: MX-NoLED, kbd_SW_Hole:SW_Hole_1u, F.Cu at (422.4, 44.2)
- added K_#8: MX-NoLED, kbd_SW_Hole:SW_Hole_1u, F.Cu at (441.5, 44.2)
- added K_#9: MX-NoLED, kbd_SW_Hole:SW_Hole_1u, F.Cu at (460.5, 44.2)
- added K_,1: MX-NoLED, kbd_SW_Hole:SW_Hole_1u, F.Cu at (460.5, 101.4)
- added K_-1: MX-NoLED, kbd_SW_Hole:SW_Hole_1u, F.Cu at (498.6, 44.2)
- added K_.1: MX-NoLED, kbd_SW_Hole:SW_Hole_1u, F.Cu at (479.6, 101.4)
- added K_/1: MX-NoLED, kbd_SW_Hole:SW_Hole_1u, F.Cu at (498.6, 101.4)
- added K_:1: MX-NoLED, kbd_SW_Hole:SW_Hole_1u, F.Cu at (512.9, 82.3)
- added K_;1: MX-NoLED, kbd_SW_Hole:SW_Hole_1u, F.Cu at (493.9, 82.3)
- added K_=1: MX-NoLED, kbd_SW_Hole:SW_Hole_1u, F.Cu at (517.7, 44.2)
- added K_@1: MX-NoLED, kbd_SW_Hole:SW_Hole_1u, F.Cu at (508.2, 63.3)
- added K_A1: MX-NoLED, kbd_SW_Hole:SW_Hole_1u, F.Cu at (322.4, 82.3)
- added K_B1: MX-NoLED, kbd_SW_Hole:SW_Hole_1u, F.Cu at (403.4, 101.4)
- added K_BKSL1: MX-NoLED, kbd_SW_Hole:SW_Hole_1u, F.Cu at (517.7, 101.4)
- added K_BKSPC1: MX-NoLED, kbd_SW_Hole:SW_Hole_1u, F.Cu at (555.8, 44.2)
- added K_C1: MX-NoLED, kbd_SW_Hole:SW_Hole_1u, F.Cu at (365.3, 101.4)
- added K_CAPS1: MX-LED, kbd_SW_Hole:SW_Hole_1.75u, F.Cu at (296.2, 82.3)
- added K_D1: MX-NoLED, kbd_SW_Hole:SW_Hole_1u, F.Cu at (360.5, 82.3)
- added K_DOWN1: MX-NoLED, kbd_SW_Hole:SW_Hole_1u, F.Cu at (536.7, 120.4)
- added K_E1: MX-NoLED, kbd_SW_Hole:SW_Hole_1u, F.Cu at (355.8, 63.3)
- added K_ENTER1: MX-NoLED, kbd_SW_Hole:SW_Hole_2u, F.Cu at (553.4, 72.8)
- added K_ESC1: MX-NoLED, kbd_SW_Hole:SW_Hole_1u, F.Cu at (289.1, 44.2)
- added K_F1: MX-NoLED, kbd_SW_Hole:SW_Hole_1u, F.Cu at (379.6, 82.3)
- added K_G1: MX-NoLED, kbd_SW_Hole:SW_Hole_1u, F.Cu at (398.6, 82.3)
- added K_H1: MX-NoLED, kbd_SW_Hole:SW_Hole_1u, F.Cu at (417.7, 82.3)
- added K_HENK1: MX-NoLED, kbd_SW_Hole:SW_Hole_1u, F.Cu at (436.7, 120.4)
- added K_I1: MX-NoLED, kbd_SW_Hole:SW_Hole_1u, F.Cu at (451.0, 63.3)
- added K_J1: MX-NoLED, kbd_SW_Hole:SW_Hole_1u, F.Cu at (436.7, 82.3)
- added K_K1: MX-NoLED, kbd_SW_Hole:SW_Hole_1u, F.Cu at (455.8, 82.3)
- added K_L1: MX-NoLED, kbd_SW_Hole:SW_Hole_1u, F.Cu at (474.8, 82.3)
- added K_LALT1: MX-NoLED, kbd_SW_Hole:SW_Hole_1u, F.Cu at (351.0, 120.4)
- added K_LCTRL1: MX-NoLED, kbd_SW_Hole:SW_Hole_1u, F.Cu at (289.1, 120.4)
- added K_LEFT1: MX-NoLED, kbd_SW_Hole:SW_Hole_1u, F.Cu at (517.7, 120.4)
- added K_LSFT1: MX-NoLED, kbd_SW_Hole:SW_Hole_2u, F.Cu at (298.6, 101.4)
- added K_LSPACE1: MX-NoLED, kbd_SW_Hole:SW_Hole_1.25u, F.Cu at (391.5, 120.4)
- added K_M1: MX-NoLED, kbd_SW_Hole:SW_Hole_1u, F.Cu at (441.5, 101.4)
- added K_N1: MX-NoLED, kbd_SW_Hole:SW_Hole_1u, F.Cu at (422.4, 101.4)
- added K_NHENK1: MX-NoLED, kbd_SW_Hole:SW_Hole_1u, F.Cu at (370.1, 120.4)
- added K_O1: MX-NoLED, kbd_SW_Hole:SW_Hole_1u, F.Cu at (470.1, 63.3)
- added K_P1: MX-NoLED, kbd_SW_Hole:SW_Hole_1u, F.Cu at (489.1, 63.3)
- added K_Q1: MX-NoLED, kbd_SW_Hole:SW_Hole_1u, F.Cu at (317.7, 63.3)
- added K_R1: MX-NoLED, kbd_SW_Hole:SW_Hole_1u, F.Cu at (374.8, 63.3)
- added K_RIGHT1: MX-NoLED, kbd_SW_Hole:SW_Hole_1u, F.Cu at (555.8, 120.4)
- added K_RSFT1: MX-NoLED, kbd_SW_Hole:SW_Hole_1u, F.Cu at (555.8, 101.4)
- added K_RSPACE1: MX-NoLED, kbd_SW_Hole:SW_Hole_1.25u, F.Cu at (415.3, 120.4)
- added K_S1: MX-NoLED, kbd_SW_Hole:SW_Hole_1u, F.Cu at (341.5, 82.3)
- added K_T1: MX-NoLED, kbd_SW_Hole:SW_Hole_1u, F.Cu at (393.9, 63.3)
- added K_TAB1: MX-NoLED, kbd_SW_Hole:SW_Hole_1.5u, F.Cu at (293.9, 63.3)
- added K_U1: MX-NoLED, kbd_SW_Hole:SW_Hole_1u, F.Cu at (432.0, 63.3)
- added K_UP1: MX-NoLED, kbd_SW_Hole:SW_Hole_1u, F.Cu at (536.7, 101.4)
- added K_V1: MX-NoLED, kbd_SW_Hole:SW_Hole_1u, F.Cu at (384.3, 101.4)
- added K_W1: MX-NoLED, kbd_SW_Hole:SW_Hole_1u, F.Cu at (336.7, 63.3)
- added K_WIN1: MX-NoLED, kbd_SW_Hole:SW_Hole_1u, F.Cu at (455.8, 120.4)
- added K_X1: MX-NoLED, kbd_SW_Hole:SW_Hole_1u, F.Cu at (346.2, 101.4)
- added K_Y1: MX-NoLED, kbd_SW_Hole:SW_Hole_1u, F.Cu at (412.9, 63.3)
- added K_YEN1: MX-NoLED, kbd_SW_Hole:SW_Hole_1u, F.Cu at (536.7, 44.2)
- added K_Z1: MX-NoLED, kbd_SW_Hole:SW_Hole_1u, F.Cu at (327.2, 101.4)
- added K_[1: MX-NoLED, kbd_SW_Hole:SW_Hole_1u, F.Cu at (527.2, 63.3)
- added K_]1: MX-NoLED, kbd_SW_Hole:SW_Hole_1u, F.Cu at (532.0, 82.3)
- K_#0_1, K_#1, K_#2, K_#3, K_#4, K_#5, K_#6, K_#7, K_#8, K_#9, K_,1, K_-1, K_.1, K_/1, K_:1, K_;1, K_=1, K_@1, K_A1, K_B1, K_BKSL1, K_BKSPC1, K_C1, K_D1, K_DOWN1, K_E1, K_ESC1, K_F1, K_G1, K_H1, K_HENK1, K_I1, K_J1, K_K1, K_L1, K_LALT1, K_LCTRL1, K_LEFT1, K_M1, K_N1, K_NHENK1, K_O1, K_P1, K_Q1, K_R1, K_RIGHT1, K_RSFT1, K_S1, K_T1, K_U1, K_UP1, K_V1, K_W1, K_WIN1, K_X1, K_Y1, K_YEN1, K_Z1, K_[1, K_]1: footprint MX_Only:MXOnly-1U-Hotswap -> kbd_SW_Hole:SW_Hole_1u
- K_CAPS1: footprint MX_Only:MXOnly-1.75U-Hotswap -> kbd_SW_Hole:SW_Hole_1.75u
- K_ENTER1: footprint MX_Only:MXOnly-ISO-ROTATED-Hotswap -> kbd_SW_Hole:SW_Hole_2u
- K_LSFT1: footprint MX_Only:MXOnly-2U-Hotswap -> kbd_SW_Hole:SW_Hole_2u
- K_LSPACE1, K_RSPACE1: footprint MX_Only:MXOnly-1.25U-Hotswap -> kbd_SW_Hole:SW_Hole_1.25u
- K_TAB1: footprint MX_Only:MXOnly-1.5U-Hotswap -> kbd_SW_Hole:SW_Hole_1.5u
- moved K_[1 149.2 mm to (278.4, 316.9)
- moved K_A1 149.2 mm to (73.6, 335.9)
- moved K_CAPS1 149.2 mm to (47.5, 335.9)
- moved K_D1 149.2 mm to (111.7, 335.9)
- moved K_E1 149.2 mm to (107.0, 316.9)
- moved K_G1 149.2 mm to (149.8, 335.9)
- moved K_I1 149.2 mm to (202.2, 316.9)
- moved K_J1 149.2 mm to (187.9, 335.9)
- moved K_K1 149.2 mm to (207.0, 335.9)
- moved K_L1 149.2 mm to (226.0, 335.9)
- moved K_Q1 149.2 mm to (68.9, 316.9)
- moved K_R1 149.2 mm to (126.0, 316.9)
- moved K_S1 149.2 mm to (92.7, 335.9)
- moved K_TAB1 149.2 mm to (45.1, 316.9)
- moved K_U1 149.2 mm to (183.2, 316.9)
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Routing:
- net COL13: track 368.3 -> 0.00 mm, vias 4 -> 0
- net ROW0: track 356.7 -> 0.00 mm, vias 2 -> 0
- net ROW1: track 342.8 -> 0.00 mm, vias 4 -> 0
- net COL12: track 306.0 -> 0.00 mm, vias 5 -> 0
- net ROW2: track 305.6 -> 0.00 mm, vias 4 -> 0
- net COL11: track 284.8 -> 0.00 mm, vias 5 -> 0
- net ROW4: track 282.7 -> 0.00 mm, vias 2 -> 0
- net COL10: track 257.0 -> 0.00 mm, vias 5 -> 0
- net ROW3: track 249.2 -> 0.00 mm
- net GND: track 241.1 -> 0.00 mm, vias 4 -> 0
- net COL9: track 238.7 -> 0.00 mm, vias 5 -> 0
- net COL7: track 227.6 -> 0.00 mm, vias 5 -> 0
- net COL8: track 220.0 -> 0.00 mm, vias 5 -> 0
- net COL6: track 208.5 -> 0.00 mm, vias 5 -> 0
- net COL5: track 186.3 -> 0.00 mm, vias 5 -> 0
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- removed copper zone on F.Cu, net (none)
- removed copper zone on B.Cu, net Earth
- removed copper zone on B.Cu, net GND
Other:
- board size 285 x 95.1 mm -> 15.9 x 30.8 mm
- board text removed: "1.25U"
- board text removed: "1.5U"
- board text removed: "1.75U"
- board text removed: "2U"
- board text removed: "D+"
- board text removed: "D-"
- board text removed: "GND"
- board text removed: "ISO-ENTER"
- board text removed: "KMKB-JP_Poker"
- board text removed: "KMKB-JP_Poker | 20230325 | Kuzumotch"
- board text removed: "RESET"
- board text removed: "VCC"

Commit message: SAVE POINT2
Parts:
- moved K_#2 152.8 mm to (187.9, 107.2)
- moved K_#3 152.8 mm to (207.0, 107.2)
- moved K_#4 152.8 mm to (226.1, 107.2)
- moved K_#6 152.8 mm to (264.1, 107.2)
- moved K_#7 152.8 mm to (283.2, 107.2)
- moved K_#8 152.8 mm to (302.2, 107.2)
- moved K_#9 152.8 mm to (321.3, 107.2)
- moved K_,1 152.8 mm to (321.3, 164.4)
- moved K_-1 152.8 mm to (359.4, 107.2)
- moved K_/1 152.8 mm to (359.4, 164.4)
- moved K_;1 152.8 mm to (354.6, 145.3)
- moved K_=1 152.8 mm to (378.4, 107.2)
- moved K_@1 152.8 mm to (368.9, 126.3)
- moved K_A1 152.8 mm to (183.2, 145.3)
- moved K_B1 152.8 mm to (264.1, 164.4)
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Other:
- board size 15.9 x 30.8 mm -> 287.7 x 215.2 mm
